File: PCB V1/PCB V1.kicad_pcb (KiCad board)
At the start: 2 copper layers, 22.9 x 46.9 mm, 9 parts, among them J2 AVR-ISP-6, U2 ATtiny45-20SU, U4 BoronV1.0

Commit message: Added project foorprints
Parts:
- U4: footprint Margo_Lib:BoronV1.0 -> ProjectFootprints:BoronV1.0
Connections:
- U4 pad 1: (no net) -> Net-(U4-Pad1)
- U4 pad 10: (no net) -> Net-(U4-Pad10)
- U4 pad 11: (no net) -> Net-(U4-Pad11)
- U4 pad 12: (no net) -> Net-(U4-Pad12)
- U4 pad 13: (no net) -> Net-(U4-Pad13)
- U4 pad 14: (no net) -> Net-(U4-Pad14)
- U4 pad 15: (no net) -> Net-(U4-Pad15)
- U4 pad 16: (no net) -> Net-(U4-Pad16)
- U4 pad 19: (no net) -> Net-(U4-Pad19)
- U4 pad 20: (no net) -> Net-(U4-Pad20)
- U4 pad 21: (no net) -> Net-(U4-Pad21)
- U4 pad 22: (no net) -> Net-(U4-Pad22)
- U4 pad 23: (no net) -> Net-(U4-Pad23)
- U4 pad 24: (no net) -> Net-(U4-Pad24)
- U4 pad 26: (no net) -> Net-(U4-Pad26)
- U4 pad 3: (no net) -> Net-(U4-Pad3)
- U4 pad 5: (no net) -> Net-(U4-Pad5)
- U4 pad 6: (no net) -> Net-(U4-Pad6)
- U4 pad 7: (no net) -> Net-(U4-Pad7)
- U4 pad 8: (no net) -> Net-(U4-Pad8)
- U4 pad 9: (no net) -> Net-(U4-Pad9)
