File: PCB V1/PCB V1.sch (KiCad schematic (older format))
At the start: 9 parts, among them J2 AVR-ISP-6, U2 ATtiny45-20SU, U4 BoronV1.0

Commit message: Added project foorprints
Parts:
- U4: footprint Margo_Lib:BoronV1.0 -> ProjectFootprints:BoronV1.0; symbol MargoGeneral:BoronV1.0 -> ProjectSymbols:BoronV1.0
Changed lines of the file:
@@
 RST
 $Comp
-L MargoGeneral:BoronV1.0 U4
+L ProjectSymbols:BoronV1.0 U4
 U 1 1 5D9840F9
 P 2100 2950
 F 0 "U4" H 2650 4815 50  0000 C CNN
 F 1 "BoronV1.0" H 2650 4724 50  0000 C CNN
-F 2 "Margo_Lib:BoronV1.0" H 1750 2650 50  0001 C CNN
+F 2 "ProjectFootprints:BoronV1.0" H 1750 2650 50  0001 C CNN
 F 3 "" H 1850 2750 50  0001 C CNN
 	1    2100 2950
